Commit message: chore

File: lidars/RS-BPearl/xacro/RS-BPearl.xacro (robot description, xacro)
@@ -18,5 +18,5 @@
       <visual>
         <geometry>
-          <mesh filename="package://hexapod_elevation_mapping/model/sensors/RS-BPearl/meshes/BPearl.STL" />
+          <mesh filename="package://gazebo_sensors/lidars/RS-BPearl/meshes/BPearl.STL" />
         </geometry>
         <origin rpy="0 -1.5708 0" xyz="0 0 0"/>

File: lidars/VLP-16/xacro/VLP-16.urdf.xacro (robot description, xacro)
@@ -18,10 +18,10 @@
       <visual>
         <geometry>
-          <mesh filename="package://hexapod_elevation_mapping/model/sensors/VLP-16/urdf/meshes/VLP16_base_1.dae" />
+          <mesh filename="package://gazebo_sensors/lidars/VLP-16/urdf/meshes/VLP16_base_1.dae" />
         </geometry>
       </visual>
       <visual>
         <geometry>
-          <mesh filename="package://hexapod_elevation_mapping/model/sensors/VLP-16/urdf/meshes/VLP16_base_2.dae" />
+          <mesh filename="package://gazebo_sensors/lidars/VLP-16/urdf/meshes/VLP16_base_2.dae" />
         </geometry>
       </visual>
@@ -47,5 +47,5 @@
         <origin xyz="0 0 -0.0377" />
         <geometry>
-          <mesh filename="package://hexapod_elevation_mapping/model/sensors/VLP-16/urdf/meshes/VLP16_scan.dae" />
+          <mesh filename="package://gazebo_sensors/lidars/VLP-16/urdf/meshes/VLP16_scan.dae" />
         </geometry>
       </visual>
